File: SirMicro3V3/SirMicro3V3.sch (KiCad schematic (older format))
At the start: 31 parts, among them J1 Conn_01x16, J2 Conn_01x16, J3 USB_B_Micro, U1 ATmega32U4-AU, U2 AP2127K-3.3, Y1 Resonator

Commit message: Board Layout Revised and 3V3 Version Added
Parts:
- added JP1: SolderJumper_2_Bridged, Jumper:SolderJumper-2_P1.3mm_Bridged_RoundedPad1.0x1.5mm, symbol Jumper:SolderJumper_2_Bridged
Connections:
- net labels added: 3V3, D10, D11, D12, D13, D4, D5, D6, D7, D8, D9, RX, SCL, SDA, TX
- net labels removed: +3.3V, IO13LED, PWRLED
- wire segments 273 -> 199
Other:
- moved on the sheet: C10, C9, ICSP6, IO13, J1, J2, PWR1, RN1, RX1, TX1, U2
