File: SirMicro3V3/SirMicro3V3.kicad_pcb (KiCad board)
At the start: 2 copper layers, 50.8 x 20.5 mm, 40 parts, among them J1 Conn_01x16, J2 Conn_01x16, J3 USB_B_Micro, U1 ATmega32U4-AU, U2 AP2127K-3.3, Y1 Resonator

Commit message: Board Layout Revised and 3V3 Version Added
Connections:
- C1 pad 1: 5V -> 3V3
- C4 pad 1: 5V -> 3V3
- C5 pad 1: 5V -> 3V3
- C7 pad 1: 5V -> 3V3
- D1 pad 1: 5V -> 3V3
- ICSP6 pad 2: 5V -> 3V3
- J1 pad 2: 5V -> 3V3
- JP1 pad 1: 5V -> 3V3
- L1 pad 1: 5V -> 3V3
- R3 pad 1: 5V -> 3V3
- RN1 pad 2: 5V -> 3V3
- U1 pad 14: 5V -> 3V3
- U1 pad 2: 5V -> 3V3
- U1 pad 34: 5V -> 3V3
- U1 pad 6: 5V -> 3V3
- U1 pad 7: 5V -> 3V3
Routing:
- net 3V3: track 6.91 -> 110.1 mm, vias 0 -> 8
- net 5V: track 120.1 -> 25.3 mm, vias 7 -> 2

Commit message: Jumper Edited
Parts:
- renumbered Y1 to 8MHz, PWR1 to PWR, RST1 to RST, RX1 to RX, TX1 to TX
