File: SirMicroDual/SirMicroDual.sch (KiCad schematic (older format))
At the start: 40 parts, among them J1 Conn_01x16, J2 Conn_01x16, J3 USB_B_Micro, Q1 Q_DUAL_PMOS_S1G1D2S2G2D1, U1 ATmega32U4-MU, U2 AP7365-W-7, U3 AZ1117-5.0, Y1 16MHz

Commit message: Part Numbers Added
Parts:
- removed R7: 68K, Resistor_SMD:R_0603_1608Metric, symbol Device:R_US
- removed R8: 22K, Resistor_SMD:R_0603_1608Metric, symbol Device:R_US
- removed U2: AP7365-W-7, Package_TO_SOT_SMD:SOT-23-5, symbol Regulator_Linear:AP2127K-ADJ
- added U2: AP2127K-3.3, Package_TO_SOT_SMD:SOT-23-5, symbol Regulator_Linear:AP2127K-3.3
- C1, C10, C7, C9: Part (none) -> C396719
- C11: Part (none) -> C7199
- C2, C3, C4, C5, C6: Part (none) -> C42998
- C8: Part (none) -> C122643
- D1: footprint Diode_SMD:D_SOD-110 -> Diode_SMD:D_SOD-123F; Part (none) -> C123900
- D2: Part (none) -> C12333
- F1: Part (none) -> C89657
- IO13: Part (none) -> C130115
- J3: Part (none) -> C132560
- L1: Part (none) -> C99366
- PWR1: Part (none) -> C130114
- Q1: value Q_DUAL_PMOS_S1G1D2S2G2D1 -> DMP2004DWK-7; Part (none) -> C332299
- R1, R2: Part (none) -> C269708
- R3, R4, R5, R6: Part (none) -> C99198
- RN1: Part (none) -> C164038
- RST1: Part (none) -> C231330
- RX1, TX1: Part (none) -> C205442
- U3: Part (none) -> C99342
- Y1: Part (none) -> C32180
Connections:
- net 3V3: now also U2.5 (VOUT)
- net 5V: now also U2.1 (VIN), U2.3 (EN)
- net GND: now also U2.2 (GND)
Changed lines of the file:
@@
 encoding utf-8
 Sheet 1 1
-Title ""
-Date ""
-Rev ""
-Comp ""
-Comment1 ""
-Comment2 ""
+Title "SirMicro"
+Date "2019-07-26"
+Rev "1"
+Comp "SirBoard"
+Comment1 "www.SirBoard.com"
+Comment2 "ATMega32U4 Based Dev Board"
 Comment3 ""
 Comment4 ""
@@
 F 2 "Connector_USB:USB_Micro-B_Molex_47346-0001" H 1800 3400 50  0001 C CNN
 F 3 "~" H 1800 3400 50  0001 C CNN
+F 4 "C132560" H 1650 3450 50  0001 C CNN "Part"
 	1    1650 3450
 	1    0    0    -1
@@
 F 2 "Capacitor_SMD:C_0805_2012Metric_Pad1.15x1.40mm_HandSolder" H 3738 4100 50  0001 C CNN
 F 3 "~" H 3700 4250 50  0001 C CNN
+F 4 "C396719" H 3700 4250 50  0001 C CNN "Part"
 	1    3700 4250
 	1    0    0    -1
@@
 F 2 "Resistor_SMD:R_0603_1608Metric" V 3440 1840 50  0001 C CNN
 F 3 "~" H 3400 1850 50  0001 C CNN
+F 4 "C99198" H 3400 1850 50  0001 C CNN "Part"
 	1    3400 1850
 	1    0    0    -1
@@
 F 2 "LED_SMD:LED_0805_2012Metric_Castellated" H 7550 4600 50  0001 C CNN
 F 3 "~" H 7550 4600 50  0001 C CNN
+F 4 "C205442" H 7550 4600 50  0001 C CNN "Part"
 	1    7550 4600
 	-1   0    0    -1
@@
 F 2 "Button_Switch_SMD:SW_SPST_B3U-1000P-B" H 2800 2500 50  0001 C CNN
 F 3 "~" H 2800 2500 50  0001 C CNN
+F 4 "C231330" H 2800 2300 50  0001 C CNN "Part"
 	1    2800 2300
 	1    0    0    -1
@@
 F 2 "Inductor_SMD:L_0805_2012Metric_Pad1.15x1.40mm_HandSolder" H 4800 1700 50  0001 C CNN
 F 3 "~" H 4800 1700 50  0001 C CNN
+F 4 "C99366" V 4800 1700 50  0001 C CNN "Part"
 	1    4800 1700
 	0    1    -1   0
@@
 F 2 "Resistor_SMD:R_0603_1608Metric" V 2640 3390 50  0001 C CNN
 F 3 "~" H 2600 3400 50  0001 C CNN
+F 4 "C269708" V 2600 3400 50  0001 C CNN "Part"
 	1    2600 3400
 	0    -1   -1   0
@@
 F 2 "Resistor_SMD:R_0603_1608Metric" V 2640 3590 50  0001 C CNN
 F 3 "~" H 2600 3600 50  0001 C CNN
+F 4 "C269708" V 2600 3600 50  0001 C CNN "Part"
 	1    2600 3600
 	0    -1   -1   0
@@
 F 2 "Capacitor_SMD:C_0603_1608Metric" H 3738 1700 50  0001 C CNN
 F 3 "~" H 3700 1850 50  0001 C CNN
+F 4 "C42998" H 3700 1850 50  0001 C CNN "Part"
 	1    3700 1850
 	1    0    0    -1
@@
 F 2 "Capacitor_SMD:C_0603_1608Metric" H 2588 1700 50  0001 C CNN
 F 3 "~" H 2550 1850 50  0001 C CNN
+F 4 "C42998" H 2550 1850 50  0001 C CNN "Part"
 	1    2550 1850
 	-1   0    0    -1
@@
 F 0 "D1" V 3054 1771 50  0000 R CNN
 F 1 "D" V 3145 1771 50  0000 R CNN
-F 2 "Diode_SMD:D_SOD-110" H 3100 1850 50  0001 C CNN
+F 2 "Diode_SMD:D_SOD-123F" H 3100 1850 50  0001 C CNN
 F 3 "~" H 3100 1850 50  0001 C CNN
+F 4 "C123900" V 3100 1850 50  0001 C CNN "Part"
 	1    3100 1850
 	0    -1   1    0
@@
 F 2 "Capacitor_SMD:C_0603_1608Metric" H 3588 3050 50  0001 C CNN
 F 3 "~" H 3550 3200 50  0001 C CNN
+F 4 "C42998" H 3550 3200 50  0001 C CNN "Part"
 	1    3550 3200
 	-1   0    0    -1
@@
 F 2 "Capacitor_SMD:C_0805_2012Metric_Pad1.15x1.40mm_HandSolder" H 5138 1750 50  0001 C CNN
 F 3 "~" H 5100 1900 50  0001 C CNN
+F 4 "C396719" H 5100 1900 50  0001 C CNN "Part"
 	1    5100 1900
 	-1   0    0    -1
@@
 F 2 "LED_SMD:LED_0805_2012Metric_Castellated" H 7550 5000 50  0001 C CNN
 F 3 "~" H 7550 5000 50  0001 C CNN
+F 4 "C205442" H 7550 5000 50  0001 C CNN "Part"
 	1    7550 5000
 	-1   0    0    -1
@@
 F 2 "LED_SMD:LED_0805_2012Metric_Castellated" H 7550 5400 50  0001 C CNN
 F 3 "~" H 7550 5400 50  0001 C CNN
+F 4 "C130114" H 7550 5400 50  0001 C CNN "Part"
 	1    7550 5400
 	-1   0    0    -1
@@
 F 2 "LED_SMD:LED_0805_2012Metric_Castellated" H 7550 5750 50  0001 C CNN
 F 3 "~" H 7550 5750 50  0001 C CNN
+F 4 "C130115" H 7550 5750 50  0001 C CNN "Part"
 	1    7550 5750
 	-1   0    0    -1
@@
 F 2 "Resistor_SMD:R_Array_Convex_4x0603" V 7175 5250 50  0001 C CNN
 F 3 "~" H 6900 5250 50  0001 C CNN
+F 4 "C164038" V 6900 5250 50  0001 C CNN "Part"
 	1    6900 5250
 	0    1    1    0
@@
 F 2 "Resistor_SMD:R_0603_1608Metric" V 5590 4540 50  0001 C CNN
 F 3 "~" H 5550 4550 50  0001 C CNN
+F 4 "C99198" V 5550 4550 50  0001 C CNN "Part"
 	1    5550 4550
 	0    -1   -1   0
@@
 F 2 "Resistor_SMD:R_1206_3216Metric" H 2050 2550 50  0001 L CNN
 F 3 "~" H 2000 2750 50  0001 C CNN
+F 4 "C89657" H 2000 2750 50  0001 C CNN "Part"
 	1    2000 2750
 	1    0    0    -1
@@
 F 2 "Capacitor_Tantalum_SMD:CP_EIA-3216-18_Kemet-A_Pad1.58x1.35mm_HandSolder" H 2238 3800 50  0001 C CNN
 F 3 "~" H 2200 3950 50  0001 C CNN
+F 4 "C122643" H 2200 3950 50  0001 C CNN "Part"
 	1    2200 3950
 	-1   0    0    -1
@@
 F 2 "Capacitor_SMD:C_0805_2012Metric_Pad1.15x1.40mm_HandSolder" H 10438 1700 50  0001 C CNN
 F 3 "~" H 10400 1850 50  0001 C CNN
+F 4 "C396719" H 10400 1850 50  0001 C CNN "Part"
 	1    10400 1850
 	-1   0    0    -1
@@
 F 2 "Capacitor_SMD:C_0805_2012Metric_Pad1.15x1.40mm_HandSolder" H 8838 1700 50  0001 C CNN
 F 3 "~" H 8800 1850 50  0001 C CNN
+F 4 "C396719" H 8800 1850 50  0001 C CNN "Part"
 	1    8800 1850
 	-1   0    0    -1
@@
 F 2 "Resistor_SMD:R_0603_1608Metric" V 2040 3940 50  0001 C CNN
 F 3 "~" H 2000 3950 50  0001 C CNN
+F 4 "C99198" H 2000 3950 50  0001 C CNN "Part"
 	1    2000 3950
 	-1   0    0    -1
@@
 F 2 "Crystal:Resonator_SMD_muRata_CSTxExxV-3Pin_3.0x1.1mm" H 3275 2750 50  0001 C CNN
 F 3 "~" H 3275 2750 50  0001 C CNN
+F 4 "C32180" V 3300 2750 50  0001 C CNN "Part"
 	1    3300 2750
 	0    1    1    0
@@
 F 2 "Capacitor_SMD:C_0603_1608Metric" H 8538 1700 50  0001 C CNN
 F 3 "~" H 8500 1850 50  0001 C CNN
+F 4 "C42998" H 8500 1850 50  0001 C CNN "Part"
 	1    8500 1850
 	-1   0    0    -1
@@
 P 6850 1650
 F 0 "Q1" V 7101 1650 50  0000 C CNN
-F 1 "Q_DUAL_PMOS_S1G1D2S2G2D1" H 7056 1605 50  0001 L CNN
+F 1 "DMP2004DWK-7" H 7056 1605 50  0001 L CNN
 F 2 "Package_TO_SOT_SMD:SOT-363_SC-70-6" H 6900 1650 50  0001 C CNN
 F 3 "~" H 6900 1650 50  0001 C CNN
+F 4 "C332299" V 6850 1650 50  0001 C CNN "Part"
 	1    6850 1650
 	0    -1   -1   0
@@
 F 2 "Capacitor_SMD:C_0603_1608Metric" H 7388 1700 50  0001 C CNN
 F 3 "~" H 7350 1850 50  0001 C CNN
+F 4 "C42998" H 7350 1850 50  0001 C CNN "Part"
 	1    7350 1850
 	-1   0    0    -1
@@
 F 2 "Resistor_SMD:R_0603_1608Metric" V 6440 1840 50  0001 C CNN
 F 3 "~" H 6400 1850 50  0001 C CNN
+F 4 "C99198" H 6400 1850 50  0001 C CNN "Part"
 	1    6400 1850
 	-1   0    0    -1
@@
 F 2 "Package_TO_SOT_SMD:SOT-143" H 1810 5450 50  0001 C CNN
 F 3 "https://assets.nexperia.com/documents/data-sheet/PRTR5V0U2X.pdf" H 1810 5450 50  0001 C CNN
+F 4 "C12333" H 1750 5450 50  0001 C CNN "Part"
 	1    1750 5450
 	1    0    0    -1
@@
 GND
 Wire Wire Line
-	10750 2150 10700 2150
-Wire Wire Line
 	7350 1700 7350 1550
 Connection ~ 7350 1550
@@
 P 7200 3100
 F 0 "Q1" H 7405 3100 50  0000 L CNN
-F 1 "Q_DUAL_PMOS_S1G1D2S2G2D1" H 7406 3055 50  0001 L CNN
+F 1 "DMP2004DWK-7" H 7406 3055 50  0001 L CNN
 F 2 "Package_TO_SOT_SMD:SOT-363_SC-70-6" H 7250 3100 50  0001 C CNN
 F 3 "~" H 7250 3100 50  0001 C CNN
+F 4 "C332299" H 7200 3100 50  0001 C CNN "Part"
 	2    7200 3100
 	0    -1   -1   0
@@
 F 2 "Capacitor_Tantalum_SMD:CP_EIA-3528-12_Kemet-T" H 7638 1700 50  0001 C CNN
 F 3 "~" H 7600 1850 50  0001 C CNN
+F 4 "C7199" H 7600 1850 50  0001 C CNN "Part"
 	1    7600 1850
 	-1   0    0    -1
@@
 $EndComp
 $Comp
-L Regulator_Linear:AP2127K-ADJ U2
-U 1 1 5E2BA0AD
-P 9500 1650
-F 0 "U2" H 9500 1990 50  0000 C CNN
-F 1 "AP7365-W-7" H 9500 1900 50  0000 C CNN
-F 2 "Package_TO_SOT_SMD:SOT-23-5" H 9500 1975 50  0001 C CNN
-F 3 "https://www.diodes.com/assets/Datasheets/AP2127.pdf" H 9500 1750 50  0001 C CNN
-	1    9500 1650
-	1    0    0    -1
-$EndComp
-$Comp
-L Device:R_US R7
-U 1 1 5E34715F
-P 10050 1300
-F 0 "R7" V 10118 1346 50  0000 L CNN
-F 1 "68K" V 10118 1255 50  0000 R CNN
-F 2 "Resistor_SMD:R_0603_1608Metric" V 10090 1290 50  0001 C CNN
-F 3 "~" H 10050 1300 50  0001 C CNN
-	1    10050 1300
-	0    -1   -1   0
-$EndComp
-$Comp
-L Device:R_US R8
-U 1 1 5E35753D
-P 10500 1300
-F 0 "R8" V 10568 1346 50  0000 L CNN
-F 1 "22K" V 10568 1255 50  0000 R CNN
-F 2 "Resistor_SMD:R_0603_1608Metric" V 10540 1290 50  0001 C CNN
-F 3 "~" H 10500 1300 50  0001 C CNN
-	1    10500 1300
-	0    -1   -1   0
-$EndComp
-Wire Wire Line
-	10250 1650 9800 1650
-Wire Wire Line
-	10200 1300 10250 1300
-Wire Wire Line
-	10650 1300 10700 1300
-Wire Wire Line
-	10700 1300 10700 2150
-Connection ~ 10700 2150
-Wire Wire Line
-	10700 2150 10400 2150
-Wire Wire Line
-	9800 1550 9850 1550
-Wire Wire Line
-	10250 1650 10250 1300
-Connection ~ 10250 1300
-Wire Wire Line
-	10250 1300 10350 1300
-Wire Wire Line
-	9900 1300 9850 1300
-Wire Wire Line
-	9850 1300 9850 1550
-Connection ~ 9850 1550
-Wire Wire Line
-	9850 1550 10400 1550
-$Comp
 L Regulator_Linear:AZ1117-5.0 U3
 U 1 1 5D85B6BD
@@
 F 2 "Package_TO_SOT_SMD:SOT-223-3_TabPin2" H 7950 1800 50  0001 C CIN
 F 3 "https://www.diodes.com/assets/Datasheets/AZ1117.pdf" H 7950 1550 50  0001 C CNN
+F 4 "C99342" H 7950 1550 50  0001 C CNN "Part"
 	1    7950 1550
 	1    0    0    -1
 $EndComp
+$Comp
+L Regulator_Linear:AP2127K-3.3 U2
+U 1 1 5E003479
+P 9500 1650
+F 0 "U2" H 9500 1990 50  0000 C CNN
+F 1 "AP2127K-3.3" H 9500 1900 50  0000 C CNN
+F 2 "Package_TO_SOT_SMD:SOT-23-5" H 9500 1975 50  0001 C CNN
+F 3 "https://www.diodes.com/assets/Datasheets/AP2127.pdf" H 9500 1750 50  0001 C CNN
+F 4 "C156285" H 9500 1650 50  0001 C CNN "Part"
+	1    9500 1650
+	1    0    0    -1
+$EndComp
+Wire Wire Line
+	10400 2150 10750 2150
+Wire Wire Line
+	9800 1550 10400 1550
 $EndSCHEMATC
