File: SirMicroV3/SirMicroV3.kicad_pcb (KiCad board)
At the start: 2 copper layers, 48.3 x 17.8 mm, 51 parts, among them J1 Conn_01x17, J2 Conn_01x17, J4 Conn_02x03_Odd_Even, U1 ATmega32U4-MU, Y1 20MHz

Commit message: Soldermask width adjusted
Other:
- rule solder_mask_min_width: 0.1 -> 0.05
Changed lines of the file:
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@@
     (pad_drill 1)
     (pad_to_mask_clearance 0)
-    (solder_mask_min_width 0.1)
+    (solder_mask_min_width 0.05)
     (aux_axis_origin 0 0)
     (grid_origin 90.17 27.94)

Commit message: SirMicroR3 Update
Silkscreen Edits
Parts:
- removed the G*** at (60.9, 35.6)
- added G***: LOGO, logo:OSHW44x31, F.Cu at (59.8, 37.7)
- added G***: LOGO, logo:logo47x67, F.Cu at (62.2, 32.7)
- moved G*** 25.2 mm to (62.1, 36.8)
- moved G*** 21.1 mm to (87.1, 36.8)
Other:
- board text added: "16MHz"
- board text added: "ATMega32U4"
- board text added: "MISO"
- board text added: "SirBoard.com"
- board text removed: "MIS"

Commit message: SirMicro Update
USB-C 3D Renders Added and Pictures Updated
Parts:
- G***: footprint logo:SirBoard112x35 -> logo:SirBoard127x40
- moved G*** 0.38 mm to (54.7, 36.8)
- moved G*** 0.09 mm to (62.0, 36.8)
